File: PCB/PCB.kicad_sch (KiCad schematic)
At the start: 79 parts, among them U1 DRV8833PWPR, U10 TPS63020, U11 TPS63020, U2 INA219AxDCN, U3 TPS22917DBV, U4 DRV8833PWP, U5 TPS22917DBV

Commit message: Error Resolutions
Parts:
- removed C11: 100n, Capacitor_SMD:C_0402_1005Metric_Pad0.74x0.62mm_HandSolder, symbol Device:C_Small
- removed JP12: Jumper_2_Small_Open, Jumper:SolderJumper-2_P1.3mm_Open_Pad1.0x1.5mm, symbol Jumper:Jumper_2_Small_Open
- removed NT1: NetTie_2, symbol Device:NetTie_2
- added C19, C20: 10u, Capacitor_SMD:C_1206_3216Metric_Pad1.33x1.80mm_HandSolder, symbol Device:C_Small
- added C21: 1u, Capacitor_SMD:C_1206_3216Metric_Pad1.33x1.80mm_HandSolder, symbol Device:C_Small
- added D3: Red, LED_SMD:LED_0603_1608Metric_Pad1.05x0.95mm_HandSolder, symbol Device:LED_Small_Filled
- added J3: Conn_02x16_Odd_Even, symbol Connector_Generic:Conn_02x16_Odd_Even
- added J4: USB_C_Receptacle_PowerOnly_6P, Nhlamolo.:USB-C-SMD_TYPE-602-T3, symbol Connector:USB_C_Receptacle_PowerOnly_6P
- added JP14, JP16: Jumper_2_Small_Open, Jumper:SolderJumper-2_P1.3mm_Open_Pad1.0x1.5mm, symbol Jumper:Jumper_2_Small_Open
- added R13: 5k6, Resistor_SMD:R_0805_2012Metric_Pad1.20x1.40mm_HandSolder, symbol Device:R_Small_US
- added R25: 1k8, Resistor_SMD:R_0603_1608Metric_Pad0.98x0.95mm_HandSolder, symbol Device:R_Small_US
- added R28, R5: 1k, Resistor_SMD:R_0402_1005Metric_Pad0.72x0.64mm_HandSolder, symbol Device:R_Small_US
- added R29: 6k8, Resistor_SMD:R_0805_2012Metric_Pad1.20x1.40mm_HandSolder, symbol Device:R_Small_US
- added R30: 10k, Resistor_SMD:R_0805_2012Metric_Pad1.20x1.40mm_HandSolder, symbol Device:R_Small_US
- added TP26, TP28, TP29, TP31, TP33: TestPoint, TestPoint:TestPoint_THTPad_D2.5mm_Drill1.2mm, symbol Connector:TestPoint
- added U12: TS5A3159ADBVR, Nhlamolo.:SOT-23-6_L2.9-W1.6-P0.95-LS2.8-BR, symbol Analog_Switch:TS5A3159ADBVR
- added U13: CH224K, Nhlamolo.:ESSOP-10_L4.9-W3.9-P1.0-LS6.0-TL-EP, symbol Interface_USB:CH224K
- added U9: TP4056-42-ESOP8, Nhlamolo.:ESOP-8_L4.9-W3.9-P1.27-LS6.0-BL-EP-1, symbol Battery_Management:TP4056-42-ESOP8
Connections:
- net 3V_VIN2 is gone; now on net Load_Supply: U11.10 (VIN2)
- net 5V Out: now also JP14.2 (B), JP16.2 (B); no longer C6.1, C7.1, R2.1, U1.1 (~{SLEEP}), U10.4 (VOUT1), U3.1 (VIN), U3.4 (CT), U4.1 (~{SLEEP}), U5.1 (VIN), U5.4 (CT)
- net CTRL_EXT_LOAD1: now also J3.25 (Pin_25)
- net CTRL_EXT_LOAD2: now also J3.7 (Pin_7)
- net EXT_LOAD1_OUT: now also C8.1, U3.5 (QOD), J3.21 (Pin_21)
- net EXT_LOAD2_OUT: now also C9.1, U5.5 (QOD), J3.11 (Pin_11)
- net GND: now also C19.2, C20.1, C21.2, J3.19 (Pin_19), J3.23 (Pin_23), J4.A12 (GND), J4.B12 (GND), R29.1, U12.4, U12.5, U13.11 (GND), U9.1 (TEMP), U9.3 (GND), U9.9 (EPAD); no longer C16.1
- net I2C1_SCL: now also J3.16 (Pin_16)
- net I2C1_SDA: now also J3.17 (Pin_17)
- net Load_Supply: now also C16.1
- net MOTOR1_A_OUT: now also J3.32 (Pin_32), TP31.1
- net MOTOR1_B_OUT: now also J3.31 (Pin_31), TP26.1
- net MOTOR1_CTRL1: now also J3.28 (Pin_28)
- net MOTOR1_CTRL2: now also J3.30 (Pin_30)
- net MOTOR2_A_OUT: now also J3.2 (Pin_2), TP29.1
- net MOTOR2_B_OUT: now also J3.1 (Pin_1), TP28.1
- net MOTOR2_CTRL1: now also J3.4 (Pin_4)
- net MOTOR2_CTRL2: now also J3.6 (Pin_6)
- net MOTOR3_A_OUT: now also J3.27 (Pin_27)
- net MOTOR3_B_OUT: now also J3.29 (Pin_29)
- net MOTOR3_CTRL1: now also J3.24 (Pin_24)
- net MOTOR3_CTRL2: now also J3.26 (Pin_26)
- net MOTOR4_A_OUT: now also J3.3 (Pin_3)
- net MOTOR4_B_OUT: now also J3.5 (Pin_5)
- net MOTOR4_CTRL1: now also J3.8 (Pin_8)
- net MOTOR4_CTRL2: now also J3.10 (Pin_10)
- net at U11.1 (VINA): now also C18.1, U11.12 (EN), U11.13 (PS/SYNC)
- net 5V_PG: now reaches U10.14 (PG)
- net 5V_PG: now also JP16.1 (A); no longer U10.5 (VOUT2)
- net at JP9.1 (A), TP24.1, U3.6 (VOUT): no longer C8.1, U3.5 (QOD)
- net at JP10.1 (A), TP25.1, U5.6 (VOUT): no longer C9.1, U5.5 (QOD)
- net 3V3 Out renamed 3V3_Out
- net 3V3_Out: now also C21.1, J3.18 (Pin_18), R28.2, U12.2, U13.1 (VDD)
- net 3V_PG renamed 3V3_PG
- net 3V_VOUT2 renamed 3V3_VOUT2
- net Switch renamed Battery
- net Battery: now also C20.2, J3.14 (Pin_14), U9.5 (BAT)
- new net: R29.2, U13.9 (CFG1)
- new net: R13.1, R25.1, U9.2 (PROG)
- new net: R25.2, U12.1
- new net: D3.1 (K), U9.7 (~{CHRG})
- new net: D3.2 (A), R5.2
- new net: R30.1, U13.8 (VBUS)
- new net: R13.2, U12.3
- new net 5V_Out: C6.1, C7.1, J3.20 (Pin_20), R2.1, TP33.1, U1.1 (~{SLEEP}), U10.4 (VOUT1), U3.1 (VIN), U3.4 (CT), U4.1 (~{SLEEP}), U5.1 (VIN), U5.4 (CT)
- new net 5V_VOUT2: JP14.1 (A), U10.5 (VOUT2)
- new net CC1: J4.A5 (CC1), U13.7 (CC1)
- new net CC2: J4.B5 (CC2), U13.6 (CC2)
- new net FAST_CHARGE_CTRL: J3.13 (Pin_13), U12.6
- new net HV-Pin: C19.1, R5.1, U9.4 (V_{CC}), U9.8 (CE)
- new net High_Voltage_(9V): J3.22 (Pin_22)
- new net VBUS: J4.A9 (VBUS), J4.B9 (VBUS), R28.1, R30.2
- no-connect marks 0 -> 10
Other:
- note added: "Charging Circuit"
- note added: "TEST: output current and output voltage"
- note added: "USb Integration"
- note removed: "TEST: output current"
- moved on the sheet: C10, C18, C6, C7, JP11, JP13, TP27

Commit message: Confirm LCSC numbers
Parts:
- removed C18: 100n, Capacitor_SMD:C_0402_1005Metric, symbol Device:C_Small
- removed JP13, JP16: Jumper_2_Small_Open, Jumper:SolderJumper-2_P1.3mm_Open_Pad1.0x1.5mm, symbol Jumper:Jumper_2_Small_Open
- removed L3: 2.2u, Inductor_SMD:L_1008_2520Metric_Pad1.43x2.20mm_HandSolder, symbol Device:L
- removed R23: 200m, Resistor_SMD:R_0603_1608Metric_Pad0.98x0.95mm_HandSolder, symbol Device:R_Small
- removed TP27: TestPoint, TestPoint:TestPoint_THTPad_D2.5mm_Drill1.2mm, symbol Connector:TestPoint
- added C11, C12: 10u, Capacitor_SMD:C_0603_1608Metric_Pad1.08x0.95mm_HandSolder, symbol Device:C_Small
- added C15: 100n, Capacitor_SMD:C_0402_1005Metric_Pad0.74x0.62mm_HandSolder, symbol Device:C_Small
- added J1: Conn_01x02_Pin, Connector_JST:JST_JWPF_B02B-JWPF-SK-R_1x02_P2.00mm_Vertical, symbol Connector:Conn_01x02_Pin
- added JP12, JP15, JP17, JP18: Jumper_2_Small_Open, Jumper:SolderJumper-2_P1.3mm_Open_Pad1.0x1.5mm, symbol Jumper:Jumper_2_Small_Open
- added L2: 2.2u, Inductor_SMD:L_1008_2520Metric_Pad1.43x2.20mm_HandSolder, symbol Device:L
- added R31: 10k, Resistor_SMD:R_0603_1608Metric_Pad0.98x0.95mm_HandSolder, symbol Device:R_Small
- added R32: 10k, Resistor_SMD:R_0805_2012Metric_Pad1.20x1.40mm_HandSolder, symbol Device:R_Small
- added R33: 0.2, Resistor_SMD:R_0603_1608Metric_Pad0.98x0.95mm_HandSolder, symbol Device:R_Small
- added R6: 10k, Resistor_SMD:R_0805_2012Metric_Pad1.20x1.40mm_HandSolder, symbol Device:R_Small_US
- added R7: 8.2k, Resistor_SMD:R_0805_2012Metric_Pad1.20x1.40mm_HandSolder, symbol Device:R_Small_US
- added TP2, TP3, TP34, TP35, TP36, TP4: TestPoint, TestPoint:TestPoint_Pad_D1.0mm, symbol Connector:TestPoint
- C13, C17: LCSC C96446 -> C96446
- C19, C20: LCSC (none) -> C13585; LSCS C13585 -> (none)
- C21: LCSC (none) -> C1848; LSCS C1848 -> (none)
- C3: LCSC C197002 -> C19702
- J3: footprint (none) -> Connector_PinHeader_2.54mm:PinHeader_2x16_P2.54mm_Vertical
- J4: footprint Nhlamolo.:USB-C-SMD_TYPE-602-T3 -> Connector_USB:USB_C_Receptacle_GCT_USB4110; LCSC (none) -> C2927028; LSCS C2927028 -> (none)
- R11: value 100 -> 200; LCSC C17408 -> C2933534
- R13: LCSC (none) -> C4382; LSCS C4382 -> (none)
- R20, R22: value 200m -> 0.2
- R21: value 200m -> 0.2; LCSC (none) -> C2286
- R25: LCSC (none) -> C4177; LSCS C4177 -> (none)
- R28: LCSC (none) -> C11702; LSCS C11702 -> (none)
- R29: LCSC (none) -> C17772; LSCS C17772 -> (none)
- R30: LCSC (none) -> C17414; LSCS C17414 -> (none)
- R4: value 560 -> 1.8k; footprint Resistor_SMD:R_0805_2012Metric_Pad1.20x1.40mm_HandSolder -> Resistor_SMD:R_0603_1608Metric; LCSC C28636 -> C4177
- TP10, TP11, TP12, TP13, TP14, TP15, TP16, TP17, TP18, TP19, TP20, TP21, TP22, TP23, TP24, TP25, TP26, TP28, TP29, TP30, TP31, TP32, TP33, TP5, TP6, TP7, TP8, TP9: footprint TestPoint:TestPoint_THTPad_D2.5mm_Drill1.2mm -> TestPoint:TestPoint_Pad_D1.0mm
- U12: LCSC (none) -> C128405; LSCS C128405 -> (none)
- U13: LCSC (none) -> C970725; LSCS C970725 -> (none)
- U3, U5: footprint Package_TO_SOT_SMD:SOT-23-6 -> Nhlamolo.:SOT-23-6_L2.9-W1.6-P0.95-LS2.8-BR; LCSC (none) -> C2681320
Connections:
- net 3V3_Out: now also JP18.2 (B), TP35.1; no longer R4.1, U11.4 (VOUT1)
- net 5V_Out: now also R4.1, JP17.1 (A); no longer TP33.1, U10.4 (VOUT1)
- net Battery: now also JP12.2 (B), TP2.1; no longer U9.5 (BAT)
- net GND: now also C11.2, C12.2, C15.2, J1.2 (Pin_2), R33.1, R7.2
- net High_Voltage_(9V): now also J4.A9 (VBUS), J4.B9 (VBUS), R28.1, R6.1, TP3.1
- net Load_Supply: now also C11.1, C12.1
- net VBUS: now also TP4.1; no longer J4.A9 (VBUS), J4.B9 (VBUS), R28.1
- net at U11.6 (L2), U11.7 (L2): now also L2.1
- net at U11.8 (L1), U11.9 (L1): now also L2.2
- net at JP5.2 (B): now also R33.2; no longer R22.2
- net at U11.1 (VINA), U11.12 (EN), U11.13 (PS/SYNC): now also C15.1
- net at JP7.2 (B): now also R22.2
- net 3V3_PG: no longer names the net of U11.14 (PG)
- net 3V3_PG: now also R32.1
- net 5V_PG: no longer names the net of U10.14 (PG)
- net 5V_PG: now also R31.1
- net HV-Pin: no longer names the net of C19.1, R5.1, U9.4 (V_{CC}), U9.8 (CE)
- net HV-Pin: now also JP15.1 (A)
- new net: JP12.1 (A), U9.5 (BAT)
- new net: JP18.1 (A), R32.2, TP36.1, U11.4 (VOUT1)
- new net: JP17.2 (B), R31.2, TP33.1, U10.4 (VOUT1)
- new net: JP15.2 (B), R6.2, R7.1, TP34.1
Other:
- moved on the sheet: C10, C19, C20, C21, D3, J3, J4, JP14, L1, R10, R13, R2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

Commit message: update
Parts:
- C11, C12: LCSC C197002 -> C19702
- C19, C20: footprint Capacitor_SMD:C_1206_3216Metric_Pad1.33x1.80mm_HandSolder -> Capacitor_SMD:C_0603_1608Metric_Pad1.08x0.95mm_HandSolder; LCSC C13585 -> C19702
Changed lines of the file:
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@@
 		(dnp no)
 		(property "Reference" "C13"
-			(at 101.6062 106.68 0)
+			(at 101.854 105.918 0)
 			(effects
 				(font
@@
 		)
 		(property "Value" "2.2u"
-			(at 104.14 109.728 0)
+			(at 104.14 106.426 0)
 			(effects
 				(font
@@
 		(dnp no)
 		(property "Reference" "C16"
-			(at 26.6762 140.97 0)
+			(at 26.416 139.192 0)
 			(effects
 				(font
@@
 		)
 		(property "Value" "2.2u"
-			(at 29.21 144.018 0)
+			(at 28.956 140.462 0)
 			(effects
 				(font
@@
 			)
 		)
-		(property "LCSC" "C197002"
+		(property "LCSC" "C19702"
 			(at 181.61 64.77 0)
 			(effects
@@
 			)
 		)
-		(property "Footprint" "Capacitor_SMD:C_1206_3216Metric_Pad1.33x1.80mm_HandSolder"
+		(property "Footprint" "Capacitor_SMD:C_0603_1608Metric_Pad1.08x0.95mm_HandSolder"
 			(at 217.17 203.2 0)
 			(effects
@@
 			)
 		)
-		(property "LCSC" "C13585"
+		(property "LCSC" "C19702"
 			(at 217.17 203.2 90)
 			(effects
@@
 			)
 		)
-		(property "Footprint" "Capacitor_SMD:C_1206_3216Metric_Pad1.33x1.80mm_HandSolder"
+		(property "Footprint" "Capacitor_SMD:C_0603_1608Metric_Pad1.08x0.95mm_HandSolder"
 			(at 240.03 222.25 0)
 			(effects
@@
 			)
 		)
-		(property "LCSC" "C13585"
+		(property "LCSC" "C19702"
 			(at 240.03 222.25 0)
 			(effects
@@
 			)
 		)
-		(property "LCSC" "C197002"
+		(property "LCSC" "C19702"
 			(at 289.56 66.04 0)
 			(effects

Commit message: Double Checking footprints and LCSC numbers
Parts:
- removed R20, R21, R22, R33: 0.2, Resistor_SMD:R_0603_1608Metric_Pad0.98x0.95mm_HandSolder, symbol Device:R_Small
- removed R26: 0, Resistor_SMD:R_0603_1608Metric_Pad0.98x0.95mm_HandSolder, symbol Device:R_Small
- removed R3: 0.22, Library:R2512, symbol Device:R_Small
- removed TP19, TP20: TestPoint, TestPoint:TestPoint_Pad_D1.0mm, symbol Connector:TestPoint
- added JP13: Jumper_3_Open, symbol Jumper:Jumper_3_Open
- added JP16: Jumper_2_Small_Open, Jumper:SolderJumper-2_P1.3mm_Open_Pad1.0x1.5mm, symbol Jumper:Jumper_2_Small_Open
- added R15, R17, R18, R19, R8, R9: 0.22, Library:R2512, symbol Device:R_Small
- added TP37, TP38: TestPoint, TestPoint:TestPoint_THTPad_D2.5mm_Drill1.2mm, symbol Connector:TestPoint
- added TP39, TP40: TestPoint, TestPoint:TestPoint_Pad_D1.0mm, symbol Connector:TestPoint
- C10, C15: footprint Capacitor_SMD:C_0402_1005Metric_Pad0.74x0.62mm_HandSolder -> Capacitor_SMD:C_0603_1608Metric_Pad1.08x0.95mm_HandSolder; LCSC C1525 -> C14663
- C13, C16, C17, C2: LCSC C96446 -> C23630
- C21: footprint Capacitor_SMD:C_1206_3216Metric_Pad1.33x1.80mm_HandSolder -> Capacitor_SMD:C_0603_1608Metric_Pad1.08x0.95mm_HandSolder; LCSC C1848 -> C5673
- C4: value 0.6u -> 1u
- R10: LCSC C2933534 -> C2933534
- R12: value 0 -> 0.22; footprint Resistor_SMD:R_0603_1608Metric_Pad0.98x0.95mm_HandSolder -> Library:R2512; LCSC C21189 -> C2960770
- R24, R27: LCSC C99782 -> C23162
- R28, R5: footprint Resistor_SMD:R_0402_1005Metric_Pad0.72x0.64mm_HandSolder -> Resistor_SMD:R_0603_1608Metric_Pad0.98x0.95mm_HandSolder; LCSC C11702 -> C21190
- R31: footprint Resistor_SMD:R_0603_1608Metric_Pad0.98x0.95mm_HandSolder -> Resistor_SMD:R_0805_2012Metric_Pad1.20x1.40mm_HandSolder
- U10, U11: footprint Package_DFN_QFN:Texas_S-PWQFN-N16_EP1.2x0.8mm_ThermalVias -> Library:TPS63020DSJR
Connections:
- net Battery: now also C4.1, U2.1 (IN+), R15.1, R8.1, R9.1, TP37.1; no longer R12.1
- net GND: now also R12.1, R17.2, R18.1, R19.2
- net Load_Supply: now also C4.2, U2.2 (IN-), JP13.2 (C), JP16.1 (A), TP38.1
- net at JP3.2 (B): now also R17.1
- net at R10.1, R2.2, U10.3 (FB): now also TP40.1
- net at R11.1, R4.2, U11.3 (FB): now also TP39.1
- net at JP5.2 (B): now also R18.2
- net at JP1.2 (B): now also R12.2
- net at JP7.2 (B): now also R19.1
- new net: JP16.2 (B), R15.2
- new net: JP13.3 (B), R9.2
- new net: JP13.1 (A), R8.2
