File: PCB/PCB.kicad_pcb (KiCad board)
At the start: 2 copper layers, 161.4 x 161.4 mm, 111 parts, among them J1 Conn_01x02_Pin, J3 Conn_02x16_Odd_Even, J4 USB_C_Receptacle_PowerOnly_6P, SW1 SW_Nidec_CAS-120A1, U1 DRV8833PWPR, U10 TPS63020, U11 TPS63020, U2 INA219AxDCN, U4 DRV8833PWP

Commit message: Dummy commit
Parts:
- removed C10, C15: 100n, Capacitor_SMD:C_0603_1608Metric_Pad1.08x0.95mm_HandSolder
- removed C11, C12, C14, C19, C22, C3, C6, C7: 10u, Capacitor_SMD:C_0603_1608Metric_Pad1.08x0.95mm_HandSolder
- removed C13, C16, C17, C2: 2.2u, Capacitor_SMD:C_0603_1608Metric_Pad1.08x0.95mm_HandSolder
- removed C21, C4: 1u, Capacitor_SMD:C_0603_1608Metric_Pad1.08x0.95mm_HandSolder
- removed C5: 0.1u, Capacitor_SMD:C_0603_1608Metric_Pad1.08x0.95mm_HandSolder
- removed C8, C9: 47u, Capacitor_SMD:C_0805_2012Metric_Pad1.18x1.45mm_HandSolder
- removed D1, D4: LED, LED_SMD:LED_0603_1608Metric_Pad1.05x0.95mm_HandSolder
- removed D3: Red, LED_SMD:LED_0603_1608Metric_Pad1.05x0.95mm_HandSolder
- removed J1: Conn_01x02_Pin, Connector_JST:JST_JWPF_B02B-JWPF-SK-R_1x02_P2.00mm_Vertical
- removed J3: Conn_02x16_Odd_Even, Connector_PinHeader_2.54mm:PinHeader_2x16_P2.54mm_Vertical
- removed J4: USB_C_Receptacle_PowerOnly_6P, Connector_USB:USB_C_Receptacle_GCT_USB4110
- removed JP1, JP10, JP11, JP14, JP15, JP16, JP17, JP18, JP19, JP2, JP21, JP22, JP23, JP24, JP3, JP4, JP5, JP6, JP7, JP8, JP9: Jumper_2_Small_Open, Jumper:SolderJumper-2_P1.3mm_Open_Pad1.0x1.5mm
- removed JP13: Jumper_3_Open, Jumper:SolderJumper-3_P1.3mm_Open_Pad1.0x1.5mm
- removed L1, L2: 2.2u, Inductor_SMD:L_1008_2520Metric_Pad1.43x2.20mm_HandSolder
- removed R10, R11: 200, Resistor_SMD:R_0805_2012Metric_Pad1.20x1.40mm_HandSolder
- removed R12, R15, R17, R18, R19, R8, R9: 0.22, Library:R2512
- removed R13: 5k6, Resistor_SMD:R_0805_2012Metric_Pad1.20x1.40mm_HandSolder
- removed R14, R16, R28, R5: 1k, Resistor_SMD:R_0603_1608Metric_Pad0.98x0.95mm_HandSolder
- removed R2, R4: 1.8k, Resistor_SMD:R_0603_1608Metric
- removed R24, R27: 4.7k, Resistor_SMD:R_0603_1608Metric_Pad0.98x0.95mm_HandSolder
- removed R25: 1k8, Resistor_SMD:R_0603_1608Metric_Pad0.98x0.95mm_HandSolder
- removed R29: 6k8, Resistor_SMD:R_0805_2012Metric_Pad1.20x1.40mm_HandSolder
- removed R30, R31, R32, R6: 10k, Resistor_SMD:R_0805_2012Metric_Pad1.20x1.40mm_HandSolder
- removed R7: 8.2k, Resistor_SMD:R_0805_2012Metric_Pad1.20x1.40mm_HandSolder
- removed SW1: SW_Nidec_CAS-120A1, Library:SW-TH_1MS1T1B1M1QES-5
- removed TP10, TP11, TP12, TP13, TP14, TP19, TP2, TP20, TP21, TP22, TP23, TP24, TP25, TP26, TP27, TP3, TP30, TP32, TP33, TP34, TP35, TP36, TP39, TP4, TP40, TP6, TP7, TP8, TP9: TestPoint, TestPoint:TestPoint_Pad_D1.0mm
- removed TP37, TP38: TestPoint, TestPoint:TestPoint_THTPad_D2.5mm_Drill1.2mm
- removed U1: DRV8833PWPR, Library:DRV8833PWPR
- removed U10, U11: TPS63020, Library:TPS63020DSJR
- removed U2: INA219AxDCN, Library:INA219AIDCNR
- removed U4: DRV8833PWP, Package_SO:HTSSOP-16-1EP_4.4x5mm_P0.65mm_EP3.4x5mm_Mask2.46x2.31mm_ThermalVias
Other:
- board outline removed
