File: PCB/_autosave-PCB.kicad_pcb (KiCad board)
At the start: 2 copper layers, 82 x 60 mm, 118 parts, among them J1 Conn_01x02_Pin, J3 Conn_02x16_Odd_Even, J4 USB_C_Receptacle_PowerOnly_6P, SW1 SW_Nidec_CAS-120A1, U1 DRV8833PWPR, U10 TPS63020, U11 TPS63020, U12 TS5A3159ADBVR, U13 CH224K, U2 INA219AxDCN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

Commit message: Dummy commit
Routing:
- net MOTOR2_CTRL2: track 0.00 -> 112.8 mm, vias 0 -> 3
Changed lines of the file:
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@@
+	)
+	(segment
+		(start 222.5 84.5)
+		(end 220.5 84.5)
+		(width 0.2)
+		(layer "F.Cu")
+		(net 34)
+	)
+	(segment
+		(start 220.5 84.5)
+		(end 220 84.5)
+		(width 0.2)
+		(layer "F.Cu")
+		(net 34)
+	)
+	(via
+		(at 220.5 84.5)
+		(size 0.6)
+		(drill 0.3)
+		(layers "F.Cu" "B.Cu")
+		(net 34)
+	)
+	(via
+		(at 222.5 84.5)
+		(size 0.6)
+		(drill 0.3)
+		(layers "F.Cu" "B.Cu")
+		(net 34)
+	)
+	(via
+		(at 220.5 84.5)
+		(size 0.6)
+		(drill 0.3)
+		(layers "F.Cu" "B.Cu")
+		(net 34)
+	)
+	(segment
+		(start 205.999 141.499)
+		(end 207 141.499)
+		(width 0.2)
+		(layer "B.Cu")
+		(net 34)
+	)
+	(segment
+		(start 223.5 137.5)
+		(end 223.5 120)
+		(width 0.2)
+		(layer "B.Cu")
+		(net 34)
+	)
+	(segment
+		(start 219.501 141.499)
+		(end 222 139)
+		(width 0.2)
+		(layer "B.Cu")
+		(net 34)
+	)
+	(segment
+		(start 223.5 88)
+		(end 224.5 87)
+		(width 0.2)
+		(layer "B.Cu")
+		(net 34)
+	)
+	(segment
+		(start 205.449 140.949)
+		(end 205.999 141.499)
+		(width 0.2)
+		(layer "B.Cu")
+		(net 34)
+	)
+	(segment
+		(start 207 141.499)
+		(end 219.501 141.499)
+		(width 0.2)
+		(layer "B.Cu")
+		(net 34)
+	)
+	(segment
+		(start 223.5 120)
+		(end 223.5 88)
+		(width 0.2)
+		(layer "B.Cu")
+		(net 34)
+	)
+	(segment
+		(start 201.52 138.5)
+		(end 202.671 137.349)
+		(width 0.2)
+		(layer "B.Cu")
+		(net 34)
+	)
+	(segment
+		(start 224.5 87)
+		(end 222.5 85)
+		(width 0.2)
+		(layer "B.Cu")
+		(net 34)
+	)
+	(segment
+		(start 222 139)
+		(end 223.5 137.5)
+		(width 0.2)
+		(layer "B.Cu")
+		(net 34)
+	)
+	(segment
+		(start 202.671 137.349)
+		(end 204.53676 137.349)
+		(width 0.2)
+		(layer "B.Cu")
+		(net 34)
+	)
+	(segment
+		(start 220.5 84.5)
+		(end 219 83)
+		(width 0.2)
+		(layer "B.Cu")
+		(net 34)
+	)
+	(segment
+		(start 219 83)
+		(end 193 83)
+		(width 0.2)
+		(layer "B.Cu")
+		(net 34)
+	)
+	(segment
+		(start 205.449 138.26124)
+		(end 205.449 140.949)
+		(width 0.2)
+		(layer "B.Cu")
+		(net 34)
+	)
+	(segment
+		(start 204.53676 137.349)
+		(end 205.449 138.26124)
+		(width 0.2)
+		(layer "B.Cu")
+		(net 34)
+	)
+	(segment
+		(start 222.5 84.5)
+		(end 222.5 84)
+		(width 0.2)
+		(layer "B.Cu")
+		(net 34)
+	)
+	(segment
+		(start 222.5 85)
+		(end 222.5 84.5)
+		(width 0.2)
+		(layer "B.Cu")
+		(net 34)
 	)
 	(segment

Commit message: Fix PCB layout
Parts:
- J1: footprint Connector_JST:JST_JWPF_B02B-JWPF-SK-R_1x02_P2.00mm_Vertical -> Connector_JST:JST_PH_S2B-PH-K_1x02_P2.00mm_Horizontal
- moved U10 233.6 mm to (176.1, 15.4), turned to 180 degrees
- moved R31 172.2 mm to (45.6, 102.0), turned to 90 degrees
- moved TP33 167.5 mm to (47.8, 93.0), turned to 90 degrees
- moved D5 166.7 mm to (55.0, 102.0)
- moved R10 164.0 mm to (52.8, 97.5)
- moved D2 163.2 mm to (57.1, 121.1), turned to -90 degrees
- moved R32 160.3 mm to (56.6, 112.0)
- moved R27 159.5 mm to (40.5, 113.1), turned to -90 degrees
- moved R24 156.3 mm to (43.5, 112.9), turned to -90 degrees
- moved C4 153.8 mm to (33.0, 112.6), turned to -90 degrees
- moved C5 150.3 mm to (36.7, 108.8)
- moved TP24 150.0 mm to (61.6, 101.5)
- moved R20 144.3 mm to (53.0, 104.5), turned to 180 degrees
- moved U3 143.2 mm to (63.6, 98.5)
- moved R19 141.4 mm to (54.1, 121.1), turned to 90 degrees
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Routing:
- net GND: track 459.7 -> 0.00 mm, vias 4 -> 0
- net Load_Supply: track 188.3 -> 0.00 mm, vias 7 -> 0
- net /5V_Out: track 158.0 -> 0.00 mm, vias 5 -> 0
- net High_Voltage_(9V): track 147.1 -> 0.00 mm, vias 7 -> 0
- net /3V3_Out: track 146.9 -> 0.00 mm, vias 5 -> 0
- net EXT_LOAD2_OUT: track 140.0 -> 0.00 mm, vias 2 -> 0
- net Net-(U10-PG): track 131.8 -> 0.00 mm, vias 2 -> 0
- net EXT_LOAD1_OUT: track 131.3 -> 0.00 mm, vias 5 -> 0
- net Net-(JP19-B): track 127.4 -> 0.00 mm, vias 7 -> 0
- net Battery: track 122.5 -> 0.00 mm, vias 4 -> 0
- net MOTOR2_CTRL2: track 112.8 -> 0.00 mm, vias 3 -> 0
- net MOTOR4_A_OUT: track 111.8 -> 0.00 mm, vias 8 -> 0
- net Net-(JP18-A): track 108.3 -> 0.00 mm, vias 4 -> 0
- net Net-(JP17-B): track 104.0 -> 0.00 mm, vias 5 -> 0
- net Net-(U13-VBUS): track 102.4 -> 0.00 mm, vias 4 -> 0
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